File: design.kicad_pcb (KiCad board)
At the start: 2 copper layers, 0 parts

Commit message: Update design.kicad_pcb
Parts:
- added C1: C_Small, Capacitor_SMD:C_0603_1608Metric, F.Cu at (172.4, 112.8)
- added C2: C_Small, Capacitor_SMD:C_0603_1608Metric, F.Cu at (177.3, 108.8)
- added J1: Conn_02x02_Counter_Clockwise, Connector_PinSocket_2.54mm:PinSocket_2x02_P2.54mm_Vertical, F.Cu at (134.8, 110.8)
- added J2: Conn_02x02_Counter_Clockwise, Connector_PinSocket_2.54mm:PinSocket_2x02_P2.54mm_Vertical, F.Cu at (160.9, 82.7)
- added J3: Conn_02x02_Counter_Clockwise, Connector_PinSocket_2.54mm:PinSocket_2x02_P2.54mm_Vertical, F.Cu at (144.4, 97.3)
- added L1: 2.2uH, Inductor_SMD:L_1008_2520Metric, F.Cu at (162.1, 109.6)
- added R1: R_Small, Resistor_SMD:R_0805_2012Metric, F.Cu at (165.5, 114.0)
- added R2: R_Small, Resistor_SMD:R_0805_2012Metric, F.Cu at (179.1, 103.9)
- added R3: R_Small, Resistor_SMD:R_0805_2012Metric, F.Cu at (184.2, 98.9)
- added TP1: TestPoint, TestPoint:TestPoint_Pad_D3.0mm, F.Cu at (167.9, 110.0)
- added TP2: TestPoint, TestPoint:TestPoint_Pad_D3.0mm, F.Cu at (174.4, 105.0)
- added TP3: TestPoint, TestPoint:TestPoint_Pad_D3.0mm, F.Cu at (160.8, 114.2)
- added TP4: TestPoint, TestPoint:TestPoint_Pad_D3.0mm, F.Cu at (174.4, 99.9)
- added TP5: TestPoint, TestPoint:TestPoint_Pad_D3.0mm, F.Cu at (169.3, 99.9)
- added TP6: TestPoint, TestPoint:TestPoint_Pad_D3.0mm, F.Cu at (179.4, 99.9)
- added TP7: TestPoint, TestPoint:TestPoint_Pad_D3.0mm, F.Cu at (169.3, 105.0)
- added TP8: RCWCTE, Snapeda:RCWCTE_TP420X150, F.Cu at (166.2, 131.7)
- added TP9: RCWCTE, Snapeda:RCWCTE_TP420X150, F.Cu at (159.9, 131.6)
- added U1: TPS63900, Package_SON:WSON-10-1EP_2.5x2.5mm_P0.5mm_EP1.2x2mm_ThermalVias, F.Cu at (172.8, 109.5)
Other:
- board outline added: 61.4 x 38.9 mm

Commit message: update
Parts:
- added J4: Conn_02x02_Counter_Clockwise, Connector_PinSocket_2.54mm:PinSocket_2x02_P2.54mm_Vertical, F.Cu at (156.7, 103.3)
- moved TP9 38.1 mm to (178.4, 98.3)
- moved J3 35.8 mm to (179.7, 103.3)
- moved J2 31.4 mm to (159.9, 114.0)
- moved TP5 30.9 mm to (144.0, 117.6)
- moved TP3 27.5 mm to (143.8, 92.6)
- moved TP2 27.2 mm to (147.4, 101.8)
- moved TP8 23.4 mm to (178.2, 111.6)
- moved TP7 22.7 mm to (188.4, 117.3)
- moved J1 19.6 mm to (153.6, 116.6), turned to -90 degrees
- moved R3 18.9 mm to (169.0, 110.2), turned to 90 degrees
- moved TP1 15.9 mm to (166.2, 94.2)
- moved R2 14.2 mm to (166.8, 111.1), turned to 90 degrees
- moved TP6 12.1 mm to (189.1, 92.7)
- moved C1 11.9 mm to (163.8, 104.6), turned to -90 degrees
- moved TP4 10.8 mm to (185.0, 101.7)
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Connections:
- J1 pad 1: Vin -> unconnected-(J1-Pad1)
- J1 pad 4: unconnected-(J1-Pad4) -> Vin
- J2 pad 1: Vin -> SEL
- J2 pad 2: SEL -> Vin
Routing:
- net Net-(L1-Pad2): track 0.00 -> 3.03 mm
- net Net-(L1-Pad1): track 0.00 -> 3.03 mm
- net GND: track 0.00 -> 1.19 mm, vias 0 -> 1
- added copper zone on B.Cu, net GND
- added copper zone on F.Cu, net GND
- added copper zone on F.Cu, net Vin
- added copper zone on F.Cu, net Vout
Other:
- board size 61.4 x 38.9 mm -> 50 x 30 mm

Commit message: update
Parts:
- TP1, TP3, TP5, TP6, TP7: value TestPoint -> GND
- TP2: value TestPoint -> Vin
- TP4: value TestPoint -> Vout
- moved R1 1.70 mm to (164.7, 111.9)
- moved R2 1.70 mm to (166.9, 112.8)
- moved R3 1.70 mm to (169.1, 111.9)
- moved J4 1.11 mm to (155.7, 103.8)
- moved TP7 0.92 mm to (189.0, 118.0), turned to 180 degrees
- moved TP8 0.82 mm to (178.4, 112.4)
- moved C2 0.45 mm to (168.8, 105.0)
- moved J2 0.45 mm to (160.1, 114.5)
- moved L1 0.45 mm to (166.4, 101.4)
- moved U1 0.45 mm to (166.4, 105.4)
- moved C1 0.45 mm to (164.0, 105.0)
- moved TP5 0.45 mm to (143.8, 118.0), turned to 180 degrees
- moved J1 0.45 mm to (153.8, 117.0)
- moved TP4 0.41 mm to (185.4, 101.6)
- moved J3 0.40 mm to (179.7, 103.8)
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Connections:
- J1 pad 1: unconnected-(J1-Pad1) -> GND
- J1 pad 3: GND -> unconnected-(J1-Pad3)
- R1 pad 1: Net-(R1-Pad1) -> GND
- R3 pad 1: Net-(R1-Pad1) -> GND
Routing:
- net Vin: track 0.00 -> 18.8 mm
- net EN: track 0.00 -> 17.5 mm
- net SEL: track 0.00 -> 12.2 mm
- net Net-(R2-Pad2): track 0.00 -> 5.28 mm
- net Net-(R1-Pad2): track 0.00 -> 5.08 mm
- net Net-(R3-Pad2): track 0.00 -> 5.08 mm
Other:
- board text added: "EN"
- board text added: "GND"
- board text added: "SEL"
- board text added: "Vin"
- board text added: "Vout"

Commit message: update
Parts:
- moved J3 2.54 mm to (179.7, 106.3), turned to -90 degrees
- moved J4 2.54 mm to (155.7, 106.3), turned to -90 degrees
- moved J2 2.54 mm to (160.1, 117.0), turned to -90 degrees
Connections:
- J2 pad 1: SEL -> GND
- J2 pad 2: Vin -> SEL
- J2 pad 3: GND -> unconnected-(J2-Pad3)
- J2 pad 4: unconnected-(J2-Pad4) -> Vin
- J3 pad 1: Vout -> GND
- J3 pad 4: GND -> Vout
- J4 pad 1: Vin -> GND
- J4 pad 4: GND -> Vin
Routing:
- net SEL: track 12.2 -> 11.2 mm
- net GND: vias 1 -> 17
Other:
- outline, holes or cut-outs redrawn
